File: source/PCB/board.sch (EAGLE design)
At the start: 36 parts, among them IC1 MEGA164P/324P/644P-AU, IC9 74LS151D, U2 UNL2003AD, U3 UNL2003AD, X1 RJ45-6L-B, X2 RJ45-6L-B, X3 RJ45-6L-B, X4 RJ45-6L-B, X5 RJ45-6L-B, X6 RJ45-6L-B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

Commit message: v2.1 files
Parts:
- added VM: (no value), pinhead:PINHD-1X3
Connections:
- new net V+: VM.2, X1.8, X2.8, X3.8, X4.8, X5.8, X6.8, X7.8, X8.8
- net +12V: now also VM.1
- net +5V: now also VM.3; no longer X1.8, X2.8, X3.8, X4.8, X5.8, X6.8, X7.8, X8.8
Changed lines of the file:
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@@
 <?xml version="1.0" encoding="utf-8"?>
 <!DOCTYPE eagle SYSTEM "eagle.dtd">
-<eagle version="7.0.0">
+<eagle version="7.3.0">
 <drawing>
 <settings>
@@
 <part name="P+5" library="supply1" deviceset="+5V" device=""/>
 <part name="GND5" library="supply1" deviceset="GND" device=""/>
-<part name="P+6" library="supply1" deviceset="+5V" device=""/>
 <part name="GND12" library="supply1" deviceset="GND" device=""/>
-<part name="P+7" library="supply1" deviceset="+5V" device=""/>
 <part name="GND13" library="supply1" deviceset="GND" device=""/>
-<part name="P+8" library="supply1" deviceset="+5V" device=""/>
 <part name="GND14" library="supply1" deviceset="GND" device=""/>
-<part name="P+9" library="supply1" deviceset="+5V" device=""/>
 <part name="GND15" library="supply1" deviceset="GND" device=""/>
-<part name="P+10" library="supply1" deviceset="+5V" device=""/>
 <part name="GND16" library="supply1" deviceset="GND" device=""/>
-<part name="P+11" library="supply1" deviceset="+5V" device=""/>
 <part name="GND17" library="supply1" deviceset="GND" device=""/>
-<part name="P+12" library="supply1" deviceset="+5V" device=""/>
 <part name="GND18" library="supply1" deviceset="GND" device=""/>
-<part name="P+13" library="supply1" deviceset="+5V" device=""/>
 <part name="GND19" library="supply1" deviceset="GND" device=""/>
 <part name="IC9" library="74xx-us" deviceset="74*151" device="D" technology="LS"/>
@@
 <part name="P+22" library="supply1" deviceset="+12V" device=""/>
 <part name="JP3" library="SparkFun-Connectors" deviceset="M02" device="PTH"/>
+<part name="P+30" library="supply1" deviceset="+12V" device=""/>
+<part name="VMOT" library="supply1" deviceset="V+" device=""/>
+<part name="P+25" library="supply1" deviceset="+5V" device=""/>
+<part name="VM" library="pinhead" deviceset="PINHD-1X3" device=""/>
+<part name="VMOT1" library="supply1" deviceset="V+" device=""/>
+<part name="VMOT2" library="supply1" deviceset="V+" device=""/>
+<part name="VMOT3" library="supply1" deviceset="V+" device=""/>
+<part name="VMOT4" library="supply1" deviceset="V+" device=""/>
+<part name="VMOT5" library="supply1" deviceset="V+" device=""/>
+<part name="VMOT6" library="supply1" deviceset="V+" device=""/>
+<part name="VMOT7" library="supply1" deviceset="V+" device=""/>
+<part name="VMOT8" library="supply1" deviceset="V+" device=""/>
 </parts>
 <sheets>
@@
 <instance part="P+5" gate="1" x="68.58" y="203.2"/>
 <instance part="GND5" gate="1" x="58.42" y="198.12"/>
-<instance part="P+6" gate="1" x="342.9" y="210.82"/>
 <instance part="GND12" gate="1" x="365.76" y="193.04"/>
-<instance part="P+7" gate="1" x="342.9" y="170.18"/>
 <instance part="GND13" gate="1" x="365.76" y="152.4"/>
-<instance part="P+8" gate="1" x="342.9" y="129.54"/>
 <instance part="GND14" gate="1" x="365.76" y="111.76"/>
-<instance part="P+9" gate="1" x="411.48" y="215.9"/>
 <instance part="GND15" gate="1" x="434.34" y="198.12"/>
-<instance part="P+10" gate="1" x="342.9" y="88.9"/>
 <instance part="GND16" gate="1" x="365.76" y="71.12"/>
-<instance part="P+11" gate="1" x="411.48" y="165.1"/>
 <instance part="GND17" gate="1" x="434.34" y="154.94"/>
-<instance part="P+12" gate="1" x="411.48" y="132.08"/>
 <instance part="GND18" gate="1" x="434.34" y="114.3"/>
-<instance part="P+13" gate="1" x="411.48" y="91.44"/>
 <instance part="GND19" gate="1" x="434.34" y="73.66"/>
 <instance part="IC9" gate="A" x="500.38" y="101.6"/>
@@
 <instance part="P+22" gate="1" x="294.64" y="149.86"/>
 <instance part="JP3" gate="G$1" x="304.8" y="91.44" rot="R180"/>
+<instance part="P+30" gate="1" x="347.98" y="251.46"/>
+<instance part="VMOT" gate="1" x="337.82" y="251.46"/>
+<instance part="P+25" gate="1" x="327.66" y="251.46"/>
+<instance part="VM" gate="A" x="312.42" y="238.76" rot="R180"/>
+<instance part="VMOT1" gate="1" x="342.9" y="210.82"/>
+<instance part="VMOT2" gate="1" x="411.48" y="215.9"/>
+<instance part="VMOT3" gate="1" x="342.9" y="170.18"/>
+<instance part="VMOT4" gate="1" x="411.48" y="165.1"/>
+<instance part="VMOT5" gate="1" x="342.9" y="129.54"/>
+<instance part="VMOT6" gate="1" x="411.48" y="132.08"/>
+<instance part="VMOT7" gate="1" x="411.48" y="91.44"/>
+<instance part="VMOT8" gate="1" x="342.9" y="88.9"/>
 </instances>
 <busses>
@@
 </segment>
 <segment>
-<wire x1="335.28" y1="198.12" x2="342.9" y2="198.12" width="0.1524" layer="91"/>
-<wire x1="342.9" y1="198.12" x2="342.9" y2="208.28" width="0.1524" layer="91"/>
-<pinref part="P+6" gate="1" pin="+5V"/>
-<pinref part="X1" gate="G$1" pin="8"/>
-</segment>
-<segment>
-<wire x1="335.28" y1="157.48" x2="342.9" y2="157.48" width="0.1524" layer="91"/>
-<wire x1="342.9" y1="157.48" x2="342.9" y2="167.64" width="0.1524" layer="91"/>
-<pinref part="P+7" gate="1" pin="+5V"/>
-<pinref part="X2" gate="G$1" pin="8"/>
-</segment>
-<segment>
-<wire x1="335.28" y1="116.84" x2="342.9" y2="116.84" width="0.1524" layer="91"/>
-<wire x1="342.9" y1="116.84" x2="342.9" y2="127" width="0.1524" layer="91"/>
-<pinref part="P+8" gate="1" pin="+5V"/>
-<pinref part="X3" gate="G$1" pin="8"/>
-</segment>
-<segment>
-<wire x1="403.86" y1="203.2" x2="411.48" y2="203.2" width="0.1524" layer="91"/>
-<wire x1="411.48" y1="203.2" x2="411.48" y2="213.36" width="0.1524" layer="91"/>
-<pinref part="P+9" gate="1" pin="+5V"/>
-<pinref part="X5" gate="G$1" pin="8"/>
-</segment>
-<segment>
-<wire x1="335.28" y1="76.2" x2="342.9" y2="76.2" width="0.1524" layer="91"/>
-<wire x1="342.9" y1="76.2" x2="342.9" y2="86.36" width="0.1524" layer="91"/>
-<pinref part="P+10" gate="1" pin="+5V"/>
-<pinref part="X4" gate="G$1" pin="8"/>
-</segment>
-<segment>
-<wire x1="403.86" y1="160.02" x2="411.48" y2="160.02" width="0.1524" layer="91"/>
-<wire x1="411.48" y1="160.02" x2="411.48" y2="162.56" width="0.1524" layer="91"/>
-<pinref part="P+11" gate="1" pin="+5V"/>
-<pinref part="X6" gate="G$1" pin="8"/>
-</segment>
-<segment>
-<wire x1="403.86" y1="119.38" x2="411.48" y2="119.38" width="0.1524" layer="91"/>
-<wire x1="411.48" y1="119.38" x2="411.48" y2="129.54" width="0.1524" layer="91"/>
-<pinref part="P+12" gate="1" pin="+5V"/>
-<pinref part="X7" gate="G$1" pin="8"/>
-</segment>
-<segment>
-<wire x1="403.86" y1="78.74" x2="411.48" y2="78.74" width="0.1524" layer="91"/>
-<wire x1="411.48" y1="78.74" x2="411.48" y2="88.9" width="0.1524" layer="91"/>
-<pinref part="P+13" gate="1" pin="+5V"/>
-<pinref part="X8" gate="G$1" pin="8"/>
-</segment>
-<segment>
 <wire x1="43.18" y1="114.3" x2="43.18" y2="111.76" width="0.1524" layer="91"/>
 <wire x1="43.18" y1="111.76" x2="43.18" y2="109.22" width="0.1524" layer="91"/>
@@
 <wire x1="175.26" y1="175.26" x2="160.02" y2="175.26" width="0.1524" layer="91"/>
 <label x="165.1" y="175.26" size="1.778" layer="95"/>
+</segment>
+<segment>
+<pinref part="VM" gate="A" pin="3"/>
+<pinref part="P+25" gate="1" pin="+5V"/>
+<wire x1="314.96" y1="241.3" x2="327.66" y2="241.3" width="0.1524" layer="91"/>
+<wire x1="327.66" y1="241.3" x2="327.66" y2="248.92" width="0.1524" layer="91"/>
 </segment>
 </net>
@@
 <junction x="294.64" y="101.6"/>
 </segment>
+<segment>
+<pinref part="VM" gate="A" pin="1"/>
+<pinref part="P+30" gate="1" pin="+12V"/>
+<wire x1="314.96" y1="236.22" x2="347.98" y2="236.22" width="0.1524" layer="91"/>
+<wire x1="347.98" y1="236.22" x2="347.98" y2="248.92" width="0.1524" layer="91"/>
+</segment>
 </net>
 <net name="LFSELA" class="0">
@@
 </segment>
 </net>
+<net name="V+" class="0">
+<segment>
+<pinref part="VMOT" gate="1" pin="V+"/>
+<wire x1="337.82" y1="248.92" x2="337.82" y2="238.76" width="0.1524" layer="91"/>
+<pinref part="VM" gate="A" pin="2"/>
+<wire x1="337.82" y1="238.76" x2="314.96" y2="238.76" width="0.1524" layer="91"/>
+</segment>
+<segment>
+<wire x1="335.28" y1="198.12" x2="342.9" y2="198.12" width="0.1524" layer="91"/>
+<wire x1="342.9" y1="198.12" x2="342.9" y2="208.28" width="0.1524" layer="91"/>
+<pinref part="X1" gate="G$1" pin="8"/>
+<pinref part="VMOT1" gate="1" pin="V+"/>
+</segment>
+<segment>
+<wire x1="403.86" y1="203.2" x2="411.48" y2="203.2" width="0.1524" layer="91"/>
+<wire x1="411.48" y1="203.2" x2="411.48" y2="213.36" width="0.1524" layer="91"/>
+<pinref part="X5" gate="G$1" pin="8"/>
+<pinref part="VMOT2" gate="1" pin="V+"/>
+</segment>
+<segment>
+<wire x1="403.86" y1="160.02" x2="411.48" y2="160.02" width="0.1524" layer="91"/>
+<wire x1="411.48" y1="160.02" x2="411.48" y2="162.56" width="0.1524" layer="91"/>
+<pinref part="X6" gate="G$1" pin="8"/>
+<pinref part="VMOT4" gate="1" pin="V+"/>
+</segment>
+<segment>
+<wire x1="335.28" y1="157.48" x2="342.9" y2="157.48" width="0.1524" layer="91"/>
+<wire x1="342.9" y1="157.48" x2="342.9" y2="167.64" width="0.1524" layer="91"/>
+<pinref part="X2" gate="G$1" pin="8"/>
+<pinref part="VMOT3" gate="1" pin="V+"/>
+</segment>
+<segment>
+<wire x1="335.28" y1="116.84" x2="342.9" y2="116.84" width="0.1524" layer="91"/>
+<wire x1="342.9" y1="116.84" x2="342.9" y2="127" width="0.1524" layer="91"/>
+<pinref part="X3" gate="G$1" pin="8"/>
+<pinref part="VMOT5" gate="1" pin="V+"/>
+</segment>
+<segment>
+<wire x1="403.86" y1="119.38" x2="411.48" y2="119.38" width="0.1524" layer="91"/>
+<wire x1="411.48" y1="119.38" x2="411.48" y2="129.54" width="0.1524" layer="91"/>
+<pinref part="X7" gate="G$1" pin="8"/>
+<pinref part="VMOT6" gate="1" pin="V+"/>
+</segment>
+<segment>
+<wire x1="403.86" y1="78.74" x2="411.48" y2="78.74" width="0.1524" layer="91"/>
+<wire x1="411.48" y1="78.74" x2="411.48" y2="88.9" width="0.1524" layer="91"/>
+<pinref part="X8" gate="G$1" pin="8"/>
+<pinref part="VMOT7" gate="1" pin="V+"/>
+</segment>
+<segment>
+<wire x1="335.28" y1="76.2" x2="342.9" y2="76.2" width="0.1524" layer="91"/>
+<wire x1="342.9" y1="76.2" x2="342.9" y2="86.36" width="0.1524" layer="91"/>
+<pinref part="X4" gate="G$1" pin="8"/>
+<pinref part="VMOT8" gate="1" pin="V+"/>
+</segment>
+</net>
