File: source/PCB/board.brd (EAGLE design)
At the start: 99.1 x 74.9 mm, 36 parts, among them IC1 MEGA164P/324P/644P-AU, IC9 74LS151D, U2 UNL2003AD, U3 UNL2003AD, X1 RJ45-6L-B, X2 RJ45-6L-B, X3 RJ45-6L-B, X4 RJ45-6L-B, X5 RJ45-6L-B, X6 RJ45-6L-B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

Commit message: v2.1 files
Parts:
- added VM: (no value), pinhead:1X03
- moved TTL_SERIAL 1.27 mm to (78.7, 25.4)
Connections:
- new net V+: VM.2, X1.8, X2.8, X3.8, X4.8, X5.8, X6.8, X7.8, X8.8
- net +12V: now also VM.1
- net +5V: now also VM.3; no longer X1.8, X2.8, X3.8, X4.8, X5.8, X6.8, X7.8, X8.8
Routing:
- net V+: track 0.00 -> 242.6 mm, vias 0 -> 4
- net GND: track 471.0 -> 535.2 mm, vias 5 -> 6
- net +5V: track 470.5 -> 423.4 mm
- net +12V: track 272.6 -> 290.3 mm
- net RX1C: track 73.9 -> 79.9 mm, vias 1 -> 2
- net SERVO2: track 111.5 -> 115.5 mm
- net SERVO5: track 113.5 -> 115.3 mm, vias 2 -> 3
- net TX1: track 200.0 -> 201.1 mm
- net RX0: track 28.2 -> 27.5 mm
- net TX0: track 26.7 -> 26.2 mm
Other:
- board text added: "12v_5v"
- board text added: "Flexostat V 2.1"
- board text added: "rev. 0"
- board text removed: "Flexostat V 2.0"
- board text removed: "rev. 1"

Commit message: updated design with mounting holes and wider traces
Parts:
- moved C7 15.4 mm to (29.8, 29.8), turned to 0 degrees
- moved C9 10.2 mm to (66.0, 57.1), turned to 0 degrees
- moved VM 3.07 mm to (91.2, 26.3), turned to 0 degrees
- moved U3 2.54 mm to (14.0, 44.5)
Routing:
- net +5V: track 423.4 -> 437.6 mm, vias 7 -> 6
- net +12V: track 290.3 -> 281.2 mm
- net V+: track 242.6 -> 235.4 mm, vias 4 -> 5
- net S8: track 10.4 -> 7.26 mm
- net GND: track 535.2 -> 532.2 mm, vias 6 -> 7
- net RX1A: track 60.1 -> 57.5 mm
- net S7: track 11.5 -> 8.96 mm
- net SERVO5: track 115.3 -> 117.9 mm
- net S9: track 8.81 -> 6.48 mm
- net SERVO2: track 115.5 -> 117.3 mm
- net RX1H: track 31.4 -> 33.0 mm
- net N$3: track 53.1 -> 54.8 mm
- net SERVO6: track 89.2 -> 90.3 mm
- net SERVO1: track 76.5 -> 77.6 mm
- net S13: track 5.95 -> 7.00 mm
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Other:
- board text added: "rev.1"
- board text removed: "rev. 0"
